File: CAO-KiCad-AMA-ESP32-Board/CAO-KiCad-AMA-ESP32-Board.kicad_sch (KiCad schematic)
At the start: 154 parts, among them J1 GPIO, J10 Conn_01x06, J11 LED, J12 EN_LED, J13 DHT Sensor, J14 Pot, J15 Select A, J16 Select B, J17 I2C, J18 VCC, J2 On/Off, J3 Conn_01x19, J4 Conn_01x19, J5 Micro_SD_Card, J6 Servo, J7 I2C, J8 5V Ext, J9 Conn_01x13, M1 Motor_Servo, Q1 IRLML6402, Q2 AO3402, SW1 SW_Push, SW2 SW_Push, SW3 SW_Push, SW4 SW_Push, SW5 SW_Push, SW6 SW_Push, SW7 RotaryEncoder_Switch_RGB, U1 ESP32-DevKitC, U2 74HC595, U3 74HC595, Y1 Crystal_GND3_Small

Commit message: Ajout du schématique et de la BOM
Parts:
- removed BZ1: Buzzer, Buzzer_Beeper:Buzzer_12x9.5RM7.6, symbol Device:Buzzer
- removed C10, C11: 10n, Capacitor_SMD:C_0805_2012Metric_Pad1.18x1.45mm_HandSolder, symbol Device:C
- removed C9: 100n, Capacitor_SMD:C_0805_2012Metric_Pad1.18x1.45mm_HandSolder, symbol Device:C
- removed D1: LED, LED_THT:LED_D3.0mm, symbol Device:LED
- removed D15, D16, D17, D18, D19, D20, D21, D22, D23, D24, D25, D26, D27, D28, D29, D30: LED, LED_SMD:LED_0805_2012Metric_Pad1.15x1.40mm_HandSolder, symbol Device:LED
- removed D2: LED_RKBG, LED_THT:LED_D5.0mm-4_RGB, symbol Device:LED_RKBG
- removed DS2, MR2, ST2: TestPoint, TestPoint:TestPoint_Pad_D2.0mm, symbol Connector:TestPoint
- removed J1: GPIO, Connector_PinHeader_2.54mm:PinHeader_1x08_P2.54mm_Vertical, symbol Connector_Generic:Conn_01x08
- removed J10: Conn_01x06, Connector_PinHeader_2.54mm:PinHeader_1x06_P2.54mm_Vertical, symbol Connector_Generic:Conn_01x06
- removed J11: LED, Connector_PinHeader_2.54mm:PinHeader_1x09_P2.54mm_Vertical, symbol Connector_Generic:Conn_01x09
- removed J12: EN_LED, Connector_PinHeader_2.54mm:PinHeader_1x02_P2.54mm_Vertical, symbol Connector_Generic:Conn_01x02
- removed J18: VCC, Connector_PinHeader_2.54mm:PinHeader_1x02_P2.54mm_Vertical, symbol Connector_Generic:Conn_01x02
- removed J2: On/Off, Connector_PinHeader_2.54mm:PinHeader_1x02_P2.54mm_Vertical, symbol Connector:Conn_01x02_Male
- removed J9: Conn_01x13, Connector_PinHeader_2.54mm:PinHeader_1x13_P2.54mm_Vertical, symbol Connector_Generic:Conn_01x13
- removed JP1: Jumper_3_Open, Jumper:SolderJumper-3_P2.0mm_Open_TrianglePad1.0x1.5mm, symbol Jumper:Jumper_3_Open
- removed M1: Motor_Servo, Connector_PinHeader_2.54mm:PinHeader_1x03_P2.54mm_Vertical, symbol Motor:Motor_Servo
- removed OE2: Jumper_2_Open, Connector_PinHeader_2.54mm:PinHeader_1x02_P2.54mm_Vertical, symbol Jumper:Jumper_2_Open
- removed Q2: AO3402, Package_TO_SOT_SMD:SOT-23, symbol Transistor_FET:AO3400A
- removed R1, R2, R3, R4: 220, Resistor_THT:R_Axial_DIN0207_L6.3mm_D2.5mm_P10.16mm_Horizontal, symbol Device:R
- removed R32, R33, R34, R35, R36, R37, R38, R39, R46, R47, R48, R50, R51, R52, R53, R54, R55, R56, R57: 560, Resistor_SMD:R_0805_2012Metric_Pad1.20x1.40mm_HandSolder, symbol Device:R
- removed R40, R41, R42, R43, R44, R45, R49, R58: 10k, Resistor_SMD:R_0805_2012Metric_Pad1.20x1.40mm_HandSolder, symbol Device:R
- removed SW7: RotaryEncoder_Switch_RGB, Divers:RotaryEncoder_Futai-24P24C-Switch-RGB_Vertical_H20mm, symbol Divers:RotaryEncoder_Switch_RGB
- removed U3: 74HC595, Package_SO:SOIC-16_3.9x9.9mm_P1.27mm, symbol 74xx:74HC595
- C12: value 10u -> DNP
- J15, J16: symbol Connector_Generic:Conn_01x03 -> Connector:Conn_01x03_Male
Connections:
- net SW Digital renamed Digital_SW
- no-connect marks 5 -> 1
Other:
- note added: "10u"
- note added: "3x LEDs utilisateur"
- note added: "=== Strapping Pins === The ESP32 chip has the following strapping pins: GPIO 0 (must be LOW to enter boot mode) GPIO 2 (must be floating or LOW during boot) GPIO 4 GPIO 5 (must be HIGH during boot) GPIO 12 (must be LOW during boot) GPIO 15 (must be HIGH during boot)"
- note added: "Commutateur analogique 5 voies"
- note added: "Commutateur digital 1 voie"
- note added: "Correspondance pour l'ADC1 : | ADC1 | GPIO | | ------ | ----- | | ADC1_CH0 | GPIO 36 | | ADC1_CH1 | GPIO 37 | | ADC1_CH2 | GPIO 38 | | ADC1_CH3 | GPIO 39 | | ADC1_CH4 | GPIO 32 | | ADC1_CH5 | GPIO 33 | | ADC1_CH6 | GPIO 34 | | ADC1_CH7 | GPIO 35 |"
- note added: "External Pull-Up Resistor"
- note added: "MPU6050"
- note added: "Modèle du module 38 broches "ESP32-WROOM-32D""
- note added: "Photorésistance (LDR)"
- note added: "Potentiomètre à glissière"
- note added: "Registre à décalage 8 bits"
- note added: "Servo Moteur"
- note added: "Support de carte micro SD"
- note added: "TODO : - Ajout de symboles pour les éléments de sérigraphie (ceux-ci disparaissent si il ne sont pas associé à un symbole) - Ajout 2x translateurs pour entrée/sortie 3V3 vers 5V sur les GPIO 16 et 17 (RX2 et TX2) - Ajout capteur piezoelectrique - Ajout encodeur rotatif - Ajout de LEDs adressables NEOPIXEL - Ajout interface DMX RS485"
- note removed: "Correspondance pour l'ADC1 | ADC1 | GPIO | | ------ | ----- | | ADC1_CH0 | GPIO 36 | | ADC1_CH1 | GPIO 37 | | ADC1_CH2 | GPIO 38 | | ADC1_CH3 | GPIO 39 | | ADC1_CH4 | GPIO 32 | | ADC1_CH5 | GPIO 33 | | ADC1_CH6 | GPIO 34 | | ADC1_CH7 | GPIO 35 |"
- note removed: "D10"
- note removed: "D11"
- note removed: "D12"
- note removed: "D13"
- note removed: "D2"
- note removed: "D3"
- note removed: "D4"
- note removed: "D5"
- note removed: "D6"
- note removed: "D7"
- note removed: "D8"
- note removed: "D9"
- note removed: "ESP32 Pin --> RGB LED : ---------------- GPIO0 --> Red GPIO2 --> Green GPI13 --> Blue"
- note removed: "NP"
- note removed: "SW Analog"
- note removed: "Shift Register Serial data input"
- note removed: "Strapping Pins The ESP32 chip has the following strapping pins: GPIO 0 (must be LOW to enter boot mode) GPIO 2 (must be floating or LOW during boot) GPIO 4 GPIO 5 (must be HIGH during boot) GPIO 12 (must be LOW during boot) GPIO 15 (must be HIGH during boot)"
- moved on the sheet: C12, C13, C3, C4, C5, C8, D10, D11, D12, D13, D14, D3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
